Commit message: Add complete Saarthi software stack
- ESP32 firmware: motor control, hall sensor odometry, watchdog, serial protocol
- ROS2 serial bridge node: UART↔ROS2, /odom publisher, TF broadcaster, fixed dual-timer race condition
- ROS2 launch file: mapping and navigation modes with conditional node loading
- Nav2 params: RPP controller, AMCL, obstacle inflation
- URDF: corrected wheel radius (0.127m) and separation (0.738m)
- FastAPI dashboard: WebSocket server, real ROS bridge + MOCK_ROS=1 mode
- Phone UI: map canvas, destination buttons, voice recognition, e-stop
- Serial test suite: 5 automated ESP32 protocol tests
- TESTING.md: 6-stage hardware integration checklist
- .gitignore: Python/ROS2/IDE artifacts

Co-Authored-By: Claude Sonnet 4.6 <noreply@anthropic.com>

File: src/wheelchair_navigation/urdf/wheelchair.urdf (robot description, URDF)
Before this commit: robot wheelchair, 7 links, 6 joints
Links:
- link left_wheel_link: geometry collision cylinder length=0.06 radius=0.127; visual cylinder length=0.06 radius=0.127
- link right_wheel_link: geometry collision cylinder length=0.06 radius=0.127; visual cylinder length=0.06 radius=0.127
Joints:
- joint left_wheel_joint: origin xyz=-0.25 0.28 -0.25 rpy=0 0 0 -> xyz=-0.25 0.369 -0.25 rpy=0 0 0
- joint right_wheel_joint: origin xyz=-0.25 -0.28 -0.25 rpy=0 0 0 -> xyz=-0.25 -0.369 -0.25 rpy=0 0 0
